File: HARDWARE/LoRa-Rev-B/LoRa_RevB.sch (KiCad schematic (older format))
At the start: 26 parts, among them CON1 CON8, CON2 CON8, U1 SX1276, X1 32.000MHz_10ppm

Commit message: Update
Other:
- note added: "8\n7\n6\n5\n4\n3\n2\n1"
- note removed: "1\n2\n3\n4\n5\n6\n7\n8"
Changed lines of the file:
@@
 EESchema Schematic File Version 4
-EELAYER 30 0
+LIBS:LoRa_RevB-cache
+EELAYER 29 0
 EELAYER END
 $Descr A4 11693 8268
@@
 Wire Wire Line
 	4600 3150 5500 3150
-Wire Bus Line
-	2300 2450 2300 4900
-Wire Bus Line
-	4300 4900 4300 6500
-Wire Bus Line
-	2300 4900 4300 4900
-Wire Bus Line
-	4650 4900 4650 6600
 Text Notes 5900 6700 0    59   ~ 0
 16\n15\n14\n13\n12\n11\n10\n9
 Text Notes 2400 6700 0    59   ~ 0
-1\n2\n3\n4\n5\n6\n7\n8
+8\n7\n6\n5\n4\n3\n2\n1
 $Bitmap
 Pos 9950 6850
@@
 EndData
 $EndBitmap
+Wire Bus Line
+	2300 2450 2300 4900
+Wire Bus Line
+	4300 4900 4300 6500
+Wire Bus Line
+	2300 4900 4300 4900
+Wire Bus Line
+	4650 4900 4650 6600
 $EndSCHEMATC
